File: week-6/gameboy less goiii/gameboy less goiii.kicad_pcb (KiCad board)
At the start: 2 copper layers, 50 x 76 mm, 20 parts, among them J1 PinSocket_01x04_P2.54mm_Verti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, J10 S4B-PH-SM4-TB, J2 S4B-PH-SM4-TB, J3 S4B-PH-SM4-TB, J7 Conn_01x07_Socket, J8 Conn_01x07_Socket, J9 S4B-PH-SM4-TB, M1 Module_XIAO-RP2040, P1 S3B-PH-SM4-TB, SW1 DOWN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

Commit message: updated
Parts:
- added J5: Screw_Terminal_01x02_P5mm, PCM_fab:TerminalBlock_OnShore_1x02_P5.00mm_Horizontal, F.Cu at (69.5, 96.0)
- C1, C2: value C_1206 -> 100nf
- R1: value R_1206 -> 1k
- moved M1 1.46 mm to (49.9, 114.9)
Routing:
- net D4: track 154.5 -> 128.3 mm
- net PWR_GND: track 346.6 -> 364.8 mm, vias 6 -> 7
- net D5: track 167.9 -> 153.6 mm
- net D3: track 46.4 -> 57.7 mm
- net PWR_5V: track 122.9 -> 130.9 mm, vias 3 -> 4
- net D7: track 19.5 -> 26.7 mm
- net BUZZER: track 90.2 -> 83.7 mm
- net D9: track 47.7 -> 43.9 mm
- net D8: track 72.1 -> 68.7 mm
- net D2: track 28.3 -> 31.7 mm
- net D1: track 27.9 -> 27.3 mm
- net D10: track 75.2 -> 75.8 mm
- net PWR_3V3: track 117.0 -> 117.5 mm

Commit message: week-9
Parts:
- added J4: PinHeader_01x04_P2.54mm_Vertical_THT_D1.4mm, PCM_fab:PinHeader_01x04_P2.54mm_Vertical_THT_D1.4mm, F.Cu at (53.8, 57.8)
Connections:
- J1 pad 3: PWR_GND -> PWR_3V3
- J1 pad 4: PWR_3V3 -> PWR_GND
Routing:
- net PWR_GND: track 364.8 -> 413.5 mm, vias 7 -> 10
- net PWR_5V: track 130.9 -> 146.0 mm, vias 4 -> 5
- net D4: track 128.3 -> 139.5 mm, vias 4 -> 5
- net D6: track 37.9 -> 27.9 mm
- net D5: track 153.6 -> 160.0 mm
- net BUZZER: track 83.7 -> 89.1 mm
- net D2: track 31.7 -> 27.5 mm
- net D8: track 68.7 -> 72.2 mm
- net PWR_3V3: track 117.5 -> 118.7 mm, vias 4 -> 5
- net D10: track 75.8 -> 76.5 mm
