File: week-6/gameboy less goiii/gameboy less goiii.kicad_sch (KiCad schematic)
At the start: 20 parts, among them J1 PinSocket_01x04_P2.54mm_Verti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, J10 S4B-PH-SM4-TB, J2 S4B-PH-SM4-TB, J3 S4B-PH-SM4-TB, J7 Conn_01x07_Socket, J8 Conn_01x07_Socket, J9 S4B-PH-SM4-TB, M1 Module_XIAO-RP2040, P1 S3B-PH-SM4-TB, SW1 DOWN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

Commit message: updated
Parts:
- added J5: Screw_Terminal_01x02_P5mm, PCM_fab:TerminalBlock_OnShore_1x02_P5.00mm_Horizontal, symbol PCM_fab:Screw_Terminal_01x02_P5mm
- C1, C2: value C_1206 -> 100nf
- R1: value R_1206 -> 1k
Connections:
- net PWR_5V: now also J5.1 (Pin_1)
- net PWR_GND: now also J5.2 (Pin_2)
Other:
- moved on the sheet: M1

Commit message: week-9
Parts:
- added J4: PinHeader_01x04_P2.54mm_Vertical_THT_D1.4mm, PCM_fab:PinHeader_01x04_P2.54mm_Vertical_THT_D1.4mm, symbol PCM_fab:PinHeader_01x04_P2.54mm_Vertical_THT_D1.4mm
Connections:
- net D4: now also J4.1 (Pin_1)
- net D5: now also J4.2 (Pin_2)
- net PWR_3V3: now also J1.3 (Pin_1), J4.3 (Pin_3); no longer J1.4 (Pin_2)
- net PWR_GND: now also J1.4 (Pin_2), J4.4 (Pin_4); no longer J1.3 (Pin_1)
