File: week-9/samd/samd.kicad_pcb (KiCad board)
At the start: 2 copper layers, 75 x 50 mm, 21 parts, among them J1 PinSocket_01x05_P2.54mm_Verti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, J10 S4B-PH-SM4-TB, J2 PinSocket_01x05_P2.54mm_Verti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, J3 PinSocket_01x05_P2.54mm_Verti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, J4 PinSocket_01x05_P2.54mm_Verti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, J5 PinSocket_01x03_P2.54mm_Verti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, J6 PinSocket_01x03_P2.54mm_Verti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, J7 S4B-PH-SM4-TB, J8 S4B-PH-SM4-TB, J9 S4B-PH-SM4-TB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

Commit message: week-9
Parts:
- moved J7 118.6 mm to (43.8, 68.0), turned to 0 degrees
- moved J8 97.7 mm to (43.5, 29.5), turned to 180 degrees
- moved J10 86.5 mm to (57.5, 68.0)
- moved J9 83.5 mm to (57.5, 29.5), turned to 180 degrees
- moved J2 53.9 mm to (106.1, 46.2)
- moved J3 53.5 mm to (106.2, 31.4), turned to 180 degrees
- moved J1 52.9 mm to (106.2, 60.6), turned to 180 degrees
- moved J4 42.0 mm to (94.2, 27.6), turned to -90 degrees
- moved P1 35.0 mm to (47.0, 48.2), turned to -90 degrees
- moved D1 30.7 mm to (60.8, 41.0), turned to 0 degrees
- moved J5 30.2 mm to (81.2, 27.6), turned to -90 degrees
- moved J6 25.8 mm to (71.0, 27.6), turned to -90 degrees
- moved 0.1uF1 25.5 mm to (74.2, 65.2), turned to 0 degrees
- moved R1 24.8 mm to (69.2, 41.0), turned to 180 degrees
- moved R2 24.1 mm to (85.0, 41.0), turned to 180 degrees
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Routing:
- net PWR_GND: track 91.9 -> 224.5 mm, vias 0 -> 2
- net PA17: track 15.5 -> 144.7 mm, vias 0 -> 3
- net VDD: track 32.3 -> 156.4 mm, vias 0 -> 4
- net PA16: track 18.2 -> 140.5 mm, vias 0 -> 2
- net V BUS: track 18.4 -> 66.5 mm
- net VDD IN: track 50.9 -> 90.5 mm, vias 4 -> 3
- net PA00: track 12.8 -> 50.4 mm
- net PA05: track 10.7 -> 47.3 mm
- net PA09: track 5.04 -> 37.6 mm, vias 0 -> 2
- net PA27: track 16.0 -> 44.8 mm
- net PA08: track 8.76 -> 37.6 mm
- net PA07: track 6.65 -> 33.8 mm
- net PA19: track 11.2 -> 37.4 mm
- net PA01: track 16.9 -> 43.0 mm, vias 0 -> 2
- net PA02: track 14.3 -> 39.6 mm
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