File: week-10/small esp 32 board/output devices.kicad_pcb (KiCad board)
At the start: 2 copper layers, 65 x 50 mm, 22 parts, among them J1 PinHeader_01x05_P2.54mm_Horiz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, J2 Screw_Terminal_01x02_P3.5mm, J3 PinHeader_01x04_P2.54mm_Horiz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, J9 Screw_Terminal_01x02_P3.5mm, SW1 Switch_Tactile_Omron, SW2 Switch_Tactile_Omron, U1 Radio_ESP32-WROOM-32E, U2 AMS1117, U3 DRV8825_STEPPER_MOTOR_DRIVER_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, U8 AMS1117

Commit message: weeks
Parts:
- added JP1: Jumper_2_Open, PCM_fab:Jumper_1206, F.Cu at (52.5, 71.8)
- J3: value PinHeader_01x04_P2.54mm_Horizontal_SMD -> motor
Changed lines of the file:
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@@
 	(net 43 "Net-(J3-Pin_1)")
 	(net 44 "Net-(J3-Pin_3)")
+	(net 45 "unconnected-(JP1-B-Pad2)")
+	(net 46 "unconnected-(JP1-A-Pad1)")
 	(footprint "PCM_fab:C_1206"
 		(layer "F.Cu")
@@
 		)
 	)
+	(footprint "PCM_fab:Jumper_1206"
+		(layer "F.Cu")
+		(at 52.55 71.75)
+		(descr "Jumper, based on SMD 1206 resistor")
+		(tags "jumper smd 1206")
+		(property "Reference" "JP1"
+			(at 0 -1.85 0)
+			(layer "F.SilkS")
+			(effects
+				(font
+					(size 1 1)
+					(thickness 0.15)
+				)
+			)
+		)
+		(property "Value" "Jumper_2_Open"
+			(at 0 1.9 0)
+			(layer "F.Fab")
+			(effects
+				(font
+					(size 1 1)
+					(thickness 0.15)
+				)
+			)
+		)
+		(property "Datasheet" "~"
+			(at 0 0 0)
+			(layer "F.Fab")
+			(hide yes)
+			(effects
+				(font
+					(size 1.27 1.27)
+					(thickness 0.15)
+				)
+			)
+		)
+		(property "Description" "Jumper, 2-pole, open"
+			(at 0 0 0)
+			(layer "F.Fab")
+			(hide yes)
+			(effects
+				(font
+					(size 1.27 1.27)
+					(thickness 0.15)
+				)
+			)
+		)
+		(property ki_fp_filters "Jumper* TestPoint*2Pads* TestPoint*Bridge*")
+		(sheetname "/")
+		(sheetfile "output devices.kicad_sch")
+		(attr smd)
+		(fp_line
+			(start -1 -1.07)
+			(end 1 -1.07)
+			(stroke
+				(width 0.12)
+				(type solid)
+			)
+			(layer "F.SilkS")
+		)
+		(fp_line
+			(start 1 1.07)
+			(end -1 1.07)
+			(stroke
+				(width 0.12)
+				(type solid)
+			)
+			(layer "F.SilkS")
+		)
+		(fp_rect
+			(start -2.7 -1.1)
+			(end 2.6 1.1)
+			(stroke
+				(width 0.05)
+				(type default)
+			)
+			(fill no)
+			(layer "F.CrtYd")
+		)
+		(fp_line
+			(start -1.6 0.8)
+			(end -1.6 -0.8)
+			(stroke
+				(width 0.1)
+				(type solid)
+			)
+			(layer "F.Fab")
+		)
+		(fp_rect
+			(start -1.55 -0.8)
+			(end 1.55 0.8)
+			(stroke
+				(width 0.1)
+				(type default)
+			)
+			(fill no)
+			(layer "F.Fab")
+		)
+		(fp_text user "${REFERENCE}"
+			(at 0 0 0)
+			(layer "F.Fab")
+			(effects
+				(font
+					(size 0.7 0.7)
+					(thickness 0.105)
+				)
+			)
+		)
+		(pad "1" smd rect
+			(at -1.7 0)
+			(size 1.4 1.7)
+			(layers "F.Cu" "F.Mask" "F.Paste")
+			(net 46 "unconnected-(JP1-A-Pad1)")
+			(pinfunction "A")
+			(pintype "passive")
+		)
+		(pad "2" smd rect
+			(at 1.7 0)
+			(size 1.4 1.7)
+			(layers "F.Cu" "F.Mask" "F.Paste")
+			(net 45 "unconnected-(JP1-B-Pad2)")
+			(pinfunction "B")
+			(pintype "passive")
+		)
+		(embedded_fonts no)
+		(model "${KICAD9_3RD_PARTY}/3dmodels/org_fabcloud_gitlab_electronics_kicad/fab.3dshapes/R_1206.step"
+			(offset
+				(xyz 0 0 0)
+			)
+			(scale
+				(xyz 1 1 1)
+			)
+			(rotate
+				(xyz 0 0 0)
+			)
+		)
+	)
 	(footprint "PCM_fab:R_1206"
 		(layer "F.Cu")
@@
 			)
 		)
-		(property "Value" "PinHeader_01x04_P2.54mm_Horizontal_SMD"
+		(property "Value" "motor"
 			(at 0 10.795 90)
 			(layer "F.Fab")
