File: week-10/small esp 32 board/output devices.kicad_sch (KiCad schematic)
At the start: 22 parts, among them J1 PinHeader_01x05_P2.54mm_Horiz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, J2 Screw_Terminal_01x02_P3.5mm, J3 PinHeader_01x04_P2.54mm_Horiz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, J9 Screw_Terminal_01x02_P3.5mm, SW1 Switch_Tactile_Omron, SW2 Switch_Tactile_Omron, U1 Radio_ESP32-WROOM-32E, U2 AMS1117, U3 DRV8825_STEPPER_MOTOR_DRIVER_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, U8 AMS1117

Commit message: weeks
Parts:
- J3: value PinHeader_01x04_P2.54mm_Horizontal_SMD -> motor
Changed lines of the file:
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@@
 	(wire
 		(pts
+			(xy 74.93 41.91) (xy 83.82 41.91)
+		)
+		(stroke
+			(width 0)
+			(type default)
+		)
+	)
+	(wire
+		(pts
 			(xy 123.19 36.83) (xy 123.19 38.1)
 		)
@@
 	(wire
 		(pts
+			(xy 73.66 44.45) (xy 83.82 44.45)
+		)
+		(stroke
+			(width 0)
+			(type default)
+		)
+	)
+	(wire
+		(pts
 			(xy 142.24 175.26) (xy 144.78 175.26)
 		)
@@
 		)
 	)
+	(wire
+		(pts
+			(xy 80.01 46.99) (xy 83.82 46.99)
+		)
+		(stroke
+			(width 0)
+			(type default)
+		)
+	)
 	(image
 		(at 427.99 129.54)
@@
 	(symbol
 		(lib_id "PCM_fab:PWR_GND")
-		(at 83.82 46.99 270)
+		(at 80.01 46.99 270)
 		(unit 1)
 		(exclude_from_sim no)
@@
 		(fields_autoplaced yes)
 		(property "Reference" "#PWR030"
-			(at 77.47 46.99 0)
+			(at 73.66 46.99 0)
 			(effects
 				(font
@@
 		)
 		(property "Value" "PWR_GND"
-			(at 80.01 46.9899 90)
+			(at 76.2 46.9899 90)
 			(effects
 				(font
@@
 		)
 		(property "Footprint" ""
-			(at 83.82 46.99 0)
+			(at 80.01 46.99 0)
 			(effects
 				(font
@@
 		)
 		(property "Datasheet" ""
-			(at 83.82 46.99 0)
+			(at 80.01 46.99 0)
 			(effects
 				(font
@@
 		)
 		(property "Description" "Power symbol creates a global label with name \"GND\" , ground"
-			(at 83.82 46.99 0)
+			(at 80.01 46.99 0)
 			(effects
 				(font
@@
 	(symbol
 		(lib_id "PCM_fab:PWR_GND")
-		(at 83.82 41.91 270)
+		(at 74.93 41.91 270)
 		(unit 1)
 		(exclude_from_sim no)
@@
 		(fields_autoplaced yes)
 		(property "Reference" "#PWR028"
-			(at 77.47 41.91 0)
+			(at 68.58 41.91 0)
 			(effects
 				(font
@@
 		)
 		(property "Value" "PWR_GND"
-			(at 80.01 41.9099 90)
+			(at 71.12 41.9099 90)
 			(effects
 				(font
@@
 		)
 		(property "Footprint" ""
-			(at 83.82 41.91 0)
+			(at 74.93 41.91 0)
 			(effects
 				(font
@@
 		)
 		(property "Datasheet" ""
-			(at 83.82 41.91 0)
+			(at 74.93 41.91 0)
 			(effects
 				(font
@@
 		)
 		(property "Description" "Power symbol creates a global label with name \"GND\" , ground"
-			(at 83.82 41.91 0)
+			(at 74.93 41.91 0)
 			(effects
 				(font
@@
 	(symbol
 		(lib_id "PCM_fab:PWR_GND")
-		(at 83.82 44.45 270)
+		(at 73.66 44.45 270)
 		(unit 1)
 		(exclude_from_sim no)
@@
 		(fields_autoplaced yes)
 		(property "Reference" "#PWR029"
-			(at 77.47 44.45 0)
+			(at 67.31 44.45 0)
 			(effects
 				(font
@@
 		)
 		(property "Value" "PWR_GND"
-			(at 80.01 44.4499 90)
+			(at 69.85 44.4499 90)
 			(effects
 				(font
@@
 		)
 		(property "Footprint" ""
-			(at 83.82 44.45 0)
+			(at 73.66 44.45 0)
 			(effects
 				(font
@@
 		)
 		(property "Datasheet" ""
-			(at 83.82 44.45 0)
+			(at 73.66 44.45 0)
 			(effects
 				(font
@@
 		)
 		(property "Description" "Power symbol creates a global label with name \"GND\" , ground"
-			(at 83.82 44.45 0)
+			(at 73.66 44.45 0)
 			(effects
 				(font
@@
 			)
 		)
-		(property "Value" "PinHeader_01x04_P2.54mm_Horizontal_SMD"
-			(at 128.27 33.02 0)
+		(property "Value" "motor"
+			(at 133.858 42.164 0)
 			(effects
 				(font
